File: Rotary Encoder with Debounce & Current Limit/rotary-encoder.sch (KiCad schematic (older format))
At the start: 20 parts, among them J1 CONN_01X05, J2 CONN_01X05, U1 74HC14

Commit message: Initial commit, v0.1
Parts:
- C1, C2, C3: value .01uF -> 0.1uF
Changed lines of the file:
@@
 P 6750 2775
 F 0 "C1" H 6775 2875 50  0000 L CNN
-F 1 ".01uF" H 6775 2675 40  0000 L CNN
+F 1 "0.1uF" H 6775 2675 40  0000 L CNN
 F 2 "BreakoutBoards:C_0603_HandSoldering" H 6788 2625 50  0001 C CNN
 F 3 "" H 6750 2775 50  0000 C CNN
@@
 P 6750 3675
 F 0 "C2" H 6775 3775 50  0000 L CNN
-F 1 ".01uF" H 6775 3575 40  0000 L CNN
+F 1 "0.1uF" H 6775 3575 40  0000 L CNN
 F 2 "BreakoutBoards:C_0603_HandSoldering" H 6788 3525 50  0001 C CNN
 F 3 "" H 6750 3675 50  0000 C CNN
@@
 P 6750 4425
 F 0 "C3" H 6775 4525 50  0000 L CNN
-F 1 ".01uF" H 6775 4325 40  0000 L CNN
+F 1 "0.1uF" H 6775 4325 40  0000 L CNN
 F 2 "BreakoutBoards:C_0603_HandSoldering" H 6788 4275 50  0001 C CNN
 F 3 "" H 6750 4425 50  0000 C CNN
